File: hardware/timer_ersatzplatine.kicad_sch (KiCad schematic)
At the start: 15 parts, among them J1 230V Netz, J2 Shelly 1PM Mini, J3 Last, J4 OLED SSD1306 0,91 Zoll, SW1 Taster T1, SW2 Taster T2, SW3 Taster T3, U1 ESP32-C3 Super Mini, U2 G3VM-601BY

Commit message: RGB-LED zähmen: I2C-SDA -> GPIO7, WS2812 (GPIO8) als gedimmte Status-LED
Die helle/warme Onboard-RGB-LED (WS2812) sitzt auf GPIO8 = bisher I2C-SDA;
der I2C-Verkehr trieb sie hell an. Lösung:
- I2C-SDA von GPIO8 auf GPIO7 verlegt (SCL bleibt GPIO9).
- WS2812 auf GPIO8 als `light: esp32_rmt_led_strip`, im 1s-Interval gesetzt:
  grün=OK, gelb=Timer laeuft, rot=Stoerung, ~8% Helligkeit (kaum Waerme).
- Konsistenz-Dreieck nachgezogen: Schaltplan-Pin GPIO8/SDA->GPIO7/SDA (Symbol
  + Instanz-Nr.), CLAUDE.md, Doku Kap. 5.1/5.2 (Netze, Pintabelle, Strapping).
- Board-Übersicht in Doku Kap. 5.2: GPIO-Belegungsgrafik (docs/img/
  board_belegung.png) + Bauteilliste des ESP32-C3 Super Mini.

Verifiziert mit `esphome compile` (ESP32-C3, Flash 56,1 %; GPIO8-Strapping-
Warnung erwartbar und unkritisch).

Co-Authored-By: Claude Opus 4.8 (1M context) <noreply@anthropic.com>
Connections:
- net SDA: now also U1.7 (GPIO7/SDA); no longer U1.8 (GPIO8/SDA)
Changed lines of the file:
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@@
     (pin "4")
     (pin "5")
-    (pin "8")
+    (pin "7")
     (pin "9")
     (instances (project "" (path "/" (reference "U1") (unit 1))))
