File: kicad-v2/Timer-Ersatzplatine-v2.kicad_sch (KiCad schematic)
At the start: 22 parts, among them J1 250-204, J2 OLED SSD1306 0,91 Zoll, J3 OLED SSD1306 0,91 Zoll, J4 OLED SSD1306 0,91 Zoll, J5 OLED SSD1306 0,91 Zoll, J6 OLED SSD1306 0,91 Zoll, K1 G3VM-601AY2, SW1 Taster T1, SW2 Taster T2, SW3 Taster T3, U1 ESP32-C3 Super Mini, X1 250-202, X2 Last, X3 Snubber, X4 Snubber

Commit message: SW4/X4 aus Schaltplan entfernt + Display 180 Grad in Firmware
- SW4 (altes On-Board-Shelly) und X4 (On-Board-Snubber) aus dem Schaltplan
  entfernt (waren nicht auf dem PCB); Schaltplan valide, 20 Komponenten.
- Display: rotation: 180 Grad in der ESPHome-Config (Montage verdreht) -
  reine Firmware-Loesung, keine Platinenaenderung, einzeilig reversibel.
- Doku-Note aktualisiert: J3-J6 bleiben als OLED-Header-Alternativen (noch
  aufs PCB zu platzieren), SW4/X4 entfernt.
- Hinweis: firmware/build/*.bin noch alter Stand -> vor Flashen neu bauen.

Co-Authored-By: Claude Opus 4.8 <noreply@anthropic.com>
Parts:
- removed SW4: (no value), Homebrew:Shelly 1PM mini, symbol Homebrew:SW_Shelly
- removed X4: Snubber, Wago 250:RC-Snubber (liegend flach), symbol 250-202:250-202
Changed lines of the file:
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@@
-	)
-	(symbol
-		(lib_id "250-202:250-202")
-		(at 220.726 155.702 0)
-		(unit 1)
-		(body_style 1)
-		(exclude_from_sim no)
-		(in_bom yes)
-		(on_board yes)
-		(in_pos_files yes)
-		(dnp no)
-		(fields_autoplaced yes)
-		(property "Reference" "X4"
-			(at 226.314 154.4319 0)
-			(show_name no)
-			(do_not_autoplace no)
-			(effects
-				(font
-					(size 1.27 1.27)
-				)
-				(justify left)
-			)
-		)
-		(property "Value" "Snubber"
-			(at 226.314 156.9719 0)
-			(show_name no)
-			(do_not_autoplace no)
-			(effects
-				(font
-					(size 1.27 1.27)
-				)
-				(justify left)
-			)
-		)
-		(property "Footprint" "Wago 250:RC-Snubber (liegend flach)"
-			(at 220.726 155.702 0)
-			(hide yes)
-			(show_name no)
-			(do_not_autoplace no)
-			(effects
-				(font
-					(size 1.27 1.27)
-				)
-				(justify bottom)
-			)
-		)
-		(property "Datasheet" ""
-			(at 220.726 155.702 0)
-			(hide yes)
-			(show_name no)
-			(do_not_autoplace no)
-			(effects
-				(font
-					(size 1.27 1.27)
-				)
-			)
-		)
-		(property "Description" "2 Position Wire to Board Terminal Block 45° (135°) Angle with Board 0.138 (3.50mm) Through Hole"
-			(at 220.726 155.702 0)
-			(hide yes)
-			(show_name no)
-			(do_not_autoplace no)
-			(effects
-				(font
-					(size 1.27 1.27)
-				)
-				(justify bottom)
-			)
-		)
-		(property "DigiKey_Part_Number" "2946-250-202-ND"
-			(at 220.726 155.702 0)
-			(hide yes)
-			(show_name no)
-			(do_not_autoplace no)
-			(effects
-				(font
-					(size 1.27 1.27)
-				)
-				(justify bottom)
-			)
-		)
-		(property "SnapEDA_Link" "https://www.snapeda.com/parts/250-202/WAGO/view-part/?ref=snap"
-			(at 220.726 155.702 0)
-			(hide yes)
-			(show_name no)
-			(do_not_autoplace no)
-			(effects
-				(font
-					(size 1.27 1.27)
-				)
-				(justify bottom)
-			)
-		)
-		(property "MF" "WAGO Innovative Connections"
-			(at 220.726 155.702 0)
-			(hide yes)
-			(show_name no)
-			(do_not_autoplace no)
-			(effects
-				(font
-					(size 1.27 1.27)
-				)
-				(justify bottom)
-			)
-		)
-		(property "Package" "None"
-			(at 220.726 155.702 0)
-			(hide yes)
-			(show_name no)
-			(do_not_autoplace no)
-			(effects
-				(font
-					(size 1.27 1.27)
-				)
-				(justify bottom)
-			)
-		)
-		(property "Check_prices" "https://www.snapeda.com/parts/250-202/WAGO/view-part/?ref=eda"
-			(at 220.726 155.702 0)
-			(hide yes)
-			(show_name no)
-			(do_not_autoplace no)
-			(effects
-				(font
-					(size 1.27 1.27)
-				)
-				(justify bottom)
-			)
-		)
-		(property "MP" "250-202"
-			(at 220.726 155.702 0)
-			(hide yes)
-			(show_name no)
-			(do_not_autoplace no)
-			(effects
-				(font
-					(size 1.27 1.27)
-				)
-				(justify bottom)
-			)
-		)
-		(pin "L1"
-		)
-		(pin "L2"
-		)
-		(instances
-			(project "Timer-Ersatzplatine"
-				(path "/6fdc0117-6431-4b50-96f7-364e63d39938"
-					(reference "X4")
-					(unit 1)
-				)
-			)
-		)
 	)
 	(symbol
@@
 					(unit 1)
 				)
-			)
-		)
-	)
-	(symbol
-		(lib_id "Homebrew:SW_Shelly")
-		(at 226.568 83.82 270)
-		(unit 1)
-		(body_style 1)
-		(exclude_from_sim no)
-		(in_bom yes)
-		(on_board yes)
-		(in_pos_files yes)
-		(dnp no)
-		(fields_autoplaced yes)
-		(property "Reference" "SW4"
-			(at 232.41 84.4549 90)
-			(show_name no)
-			(do_not_autoplace no)
-			(effects
-				(font
-					(size 1.27 1.27)
-				)
-				(justify left)
-			)
-		)
-		(property "Value" ""
-			(at 226.568 83.82 0)
-			(show_name no)
-			(do_not_autoplace no)
-			(effects
-				(font
-					(size 1.27 1.27)
-				)
-			)
-		)
-		(property "Footprint" "Homebrew:Shelly 1PM mini"
-			(at 226.568 83.82 0)
-			(hide yes)
-			(show_name no)
-			(do_not_autoplace no)
-			(effects
-				(font
-					(size 1.27 1.27)
-				)
-			)
-		)
-		(property "Datasheet" ""
-			(at 226.568 83.82 0)
-			(hide yes)
-			(show_name no)
-			(do_not_autoplace no)
-			(effects
-				(font
-					(size 1.27 1.27)
-				)
-			)
-		)
-		(property "Description" ""
-			(at 226.568 83.82 0)
-			(hide yes)
-			(show_name no)
-			(do_not_autoplace no)
-			(effects
-				(font
-					(size 1.27 1.27)
-				)
-			)
-		)
-		(pin "3"
-		)
-		(pin "1"
-		)
-		(pin "2"
-		)
-		(pin "4"
-		)
-		(instances
-			(project "Timer-Ersatzplatine"
-				(path "/6fdc0117-6431-4b50-96f7-364e63d39938"
-					(reference "SW4")
-					(unit 1)
-				)
