File: kicad-v2/Timer-Ersatzplatine-v2.kicad_pcb (KiCad board)
At the start: 4 copper layers, 101.5 x 77.4 mm, 24 parts, among them J1 250-204, J2 OLED SSD1306 0,91 Zoll, J3 OLED SSD1306 0,91 Zoll, J4 OLED SSD1306 0,91 Zoll, J5 OLED SSD1306 0,91 Zoll, J6 OLED SSD1306 0,91 Zoll, K1 G3VM-601AY2, SW1 Taster T1, SW2 Taster T2, SW3 Taster T3, U1 ESP32-C3 Super Mini, X1 Netz, X2 Last, X3 Snubber

Commit message: Fix: ESP-GND war nicht angebunden (Pad "GND" vs. Symbol-Pin-Nr. "G")
Am ESP kam keine Masse an: Der ESP32-C3-Footprint hatte das Ground-Pad "GND"
benannt, das Symbol jedoch die Pin-NUMMER "G". KiCad mappt Pin-Nummer -> Pad-Name,
"G" != "GND" -> das GND-Pad blieb ohne Netz (die Masseflaechen gossen mit Abstand
darum herum). Der ESP lief daher nur per USB (dort liefert das Kabel die Masse).

Fix: Footprint-Pad an die Symbol-Pin-Nummer angeglichen ("GND" -> "G", in
ESP32-C3-SuperMini.pretty UND im Board), Pad aufs GND-Netz gelegt, Zonen neu
gefuellt. Pad sitzt in allen 4 Masseflaechen -> bondet direkt.
Verifiziert: U1.G auf GND, DRC 0 unverbundene Elemente.

Co-Authored-By: Claude Opus 4.8 <noreply@anthropic.com>
Connections:
- PS1 pad 3: /+5V -> GND
- PS1 pad 4: GND -> /+5V
Routing:
- net /+5V: track 114.9 -> 130.1 mm
- net GND: track 173.8 -> 171.0 mm
Other:
- board text added: "+"
- board text added: "+Vo"
- board text added: "-Vo"
- board text added: "Feeder-Relais V2.0.2"
- board text removed: "Feeder-Relais V2.0.1"
Changed lines of the file:
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@@
 		)
 		(property "Value" "TSP-05 (5V/3W)"
-			(at 34.417 2.794 90)
+			(at 14.431 9.103 0)
 			(layer "B.SilkS")
 			(effects
@@
 			(layers "*.Cu" "*.Mask")
 			(remove_unused_layers no)
-			(net "/+5V")
+			(net "GND")
 			(pinfunction "+5V_3")
 			(pintype "passive")
@@
 			(layers "*.Cu" "*.Mask")
 			(remove_unused_layers no)
-			(net "GND")
+			(net "/+5V")
 			(pinfunction "GND_4")
 			(pintype "passive")
@@
 			(remove_unused_layers no)
 		)
-		(pad "GND" thru_hole circle
+		(pad "G" thru_hole circle
 			(at 7.62 6.35 90)
 			(size 1.14 1.14)
@@
 			(layers "*.Cu" "*.Mask")
 			(remove_unused_layers no)
+			(net "GND")
 		)
 		(embedded_fonts no)
@@
 		(layer "F.Fab")
 	)
-	(gr_text "Feeder-Relais V2.0.1"
+	(gr_text "Feeder-Relais V2.0.2"
 		(at 109.601 90.043 90)
 		(layer "F.SilkS")
@@
 		)
 	)
-	(gr_text "Feeder-Relais V2.0.1"
+	(gr_text "Feeder-Relais V2.0.2"
 		(at 109.474 73.787 90)
 		(layer "B.SilkS")
@@
 		)
 	)
+	(gr_text "-Vo"
+		(at 110.9 107.9 0)
+		(layer "B.SilkS")
+		(effects
+			(font
+				(size 1.5 1.5)
+				(thickness 0.25)
+			)
+			(justify mirror)
+		)
+	)
+	(gr_text "+Vo"
+		(at 120.5 122.9 0)
+		(layer "B.SilkS")
+		(effects
+			(font
+				(size 1.5 1.5)
+				(thickness 0.25)
+			)
+			(justify mirror)
+		)
+	)
+	(gr_text "+"
+		(at 176.2 52.6 0)
+		(layer "B.SilkS")
+		(effects
+			(font
+				(size 1.5 1.5)
+				(thickness 0.25)
+			)
+			(justify mirror)
+		)
+	)
 	(gr_text "TSP-05"
 		(at 131.953 119.634 0)
@@
 	)
 	(segment
-		(start 117.351 122.903)
-		(end 118.5011 122.903)
-		(width 0.2)
-		(layer "B.Cu")
-		(net "GND")
-	)
-	(segment
 		(start 181.991 96.266)
 		(end 181.991 76.073)
@@
 	)
 	(segment
-		(start 118.5011 122.903)
-		(end 129.4059 111.9982)
+		(start 185.4926 72.5714)
+		(end 182.88 75.184)
 		(width 0.2)
 		(layer "B.Cu")
@@
 	)
 	(segment
-		(start 185.4926 72.5714)
-		(end 182.88 75.184)
+		(start 117.35 107.9)
+		(end 125.31 107.9)
 		(width 0.2)
 		(layer "B.Cu")
@@
 	)
 	(segment
+		(start 125.31 107.9)
+		(end 129.41 112)
+		(width 0.2)
+		(layer "B.Cu")
+		(net "GND")
+	)
+	(segment
 		(start 129.4059 90.5316)
 		(end 130.2684 89.6691)
@@
 	)
 	(segment
+		(start 117.35 122.9)
+		(end 118.9 121.35)
+		(width 0.2)
+		(layer "F.Cu")
+		(net "/+5V")
+	)
+	(segment
 		(start 187.091 52.598)
 		(end 180.467 52.598)
@@
 	)
 	(segment
-		(start 118.133 106.6029)
-		(end 117.351 106.6029)
+		(start 118.9 121.35)
+		(end 118.9 107.37)
 		(width 0.2)
 		(layer "F.Cu")
@@
 	)
 	(segment
-		(start 117.351 107.903)
-		(end 117.351 106.6029)
+		(start 118.9 107.37)
+		(end 118.13 106.6)
 		(width 0.2)
 		(layer "F.Cu")
