File: kicad-v3/Timer-Ersatzplatine-v3.kicad_pcb (KiCad board)
At the start: 4 copper layers, 101.5 x 77.4 mm, 20 parts, among them J1 250-204, J4 OLED SSD1306 0,91 Zoll, K1 G3VM-601AY2, SW1 Taster T1, SW2 Taster T2, SW3 Taster T3, U1 ESP32-C3 Super Mini, X1 Netz, X2 Last, X3 Snubber

Commit message: v3.0.1: K1 3/4-Tausch, 230V auf Innenlagen, J4-Drehung (GND unten)
Aufbauend auf v3.0.0 (Re-Layout + Umbenennung), Board-Feinschliff:
- K1 (PhotoMOS) Pin 3/4 getauscht (Schaltplan + Board) -> L_F via-los geroutet
- Alle 230V-Bahnen auf Innenlagen verschoben: F.Cu->In1, B.Cu->In2
  (Aussenflaechen 230V-frei/beruehrsicher; GND-Zonen identisch, DRC sauber)
- J4 (OLED-Header) um 180 Grad gedreht: GND jetzt unten zu PS1;
  Reihenfolge GND/VCC/SCL/SDA, neu geroutet, GND-Zone um J4.1 ergaenzt
- Schwachstrom-Bahnen + Silk (Nutzer-GUI) nachgezogen
- DRC: 0 unverbunden, 0 Clearance/Kriechstrecke/Short (nur kosmetische Silk)
- FW_VERSION 3.0.0 -> 3.0.1; firmware/build/ neu kompiliert

Finale GUI-DRC-Kriechstreckenpruefung (K1-Waiver) durch Nutzer erfolgt.

Co-Authored-By: Claude Opus 4.8 <noreply@anthropic.com>
Parts:
- moved J4 7.62 mm to (139.6, 99.1), turned to 180 degrees
- moved F1 5.03 mm to (166.0, 110.5), turned to 90 degrees
Connections:
- K1 pad 3: /SW_SHELLY -> /L_F
- K1 pad 4: /L_F -> /SW_SHELLY
Routing:
- net GND: track 133.1 -> 86.0 mm
- net /L_F: track 85.0 -> 77.3 mm, vias 2 -> 0
- net /+3V3: track 44.3 -> 51.2 mm
- net /PMOS_DRV: track 52.5 -> 59.0 mm
- net /SW_SHELLY: track 26.3 -> 32.6 mm
- net /SDA: track 30.1 -> 24.9 mm
- net /+5V: track 130.1 -> 135.3 mm
- net /L_IN: track 15.7 -> 12.8 mm
- net /SCL: track 23.5 -> 21.6 mm
- net /O_LAST: track 53.0 -> 54.0 mm
Other:
- board text added: "Feeder-Relais V3.0.1"
- board text removed: "Feeder-Relais V2.0.2"

Commit message: v3.0.3: PS1-Polaritaet korrigiert (+5V/GND) + Routen-Feinschliff
Board-Korrektur (kritisch):
- PS1 (TSP-05) DC-Ausgang richtiggestellt: PS1.3 = GND (-Vo, Mitte),
  PS1.4 = +5V (+Vo, Rand) -- deckungsgleich mit Modul-Pinout, Silkscreen
  UND Schaltplan. In v3.0.0 war die Polaritaet versehentlich gedreht worden.
- +5V rechts an der Rand-Aussparung vorbei zu PS1.4 (+Vo) gefuehrt; +5V -> U1.5V.
- Einige Schwachstrom-Routen nachkorrigiert (Nutzer, GUI).
- DRC: 0 unverbunden, 0 Clearance/Kriechstrecke/Short/Randabstand.
- Gerber (4-lagig) neu aus dem korrigierten Board.
- FW_VERSION 3.0.2 -> 3.0.3 (Versions-Bump; Firmware funktional = 3.0.2).

Co-Authored-By: Claude Opus 4.8 <noreply@anthropic.com>
Connections:
- PS1 pad 3: /+5V -> GND
- PS1 pad 4: GND -> /+5V
Routing:
- net /+5V: track 135.3 -> 150.3 mm
- net /PMOS_DRV: track 59.0 -> 62.1 mm
- net /SDA: track 24.9 -> 27.6 mm
- net /SCL: track 21.6 -> 23.4 mm
